File: LEDDRIVE.kicad_sch (KiCad schematic)
At the start: 6 parts, among them Q1 TIP120, Q2 TIP120

Commit message: Add files via upload
Parts:
- removed D1: D, symbol Device:D
- added J1, J2: Conn_01x02_Pin, Connector_PinHeader_2.54mm:PinHeader_1x02_P2.54mm_Horizontal, symbol Connector:Conn_01x02_Pin
- added Q3, Q4: TIP120, Package_TO_SOT_THT:TO-220-3_Horizontal_TabDown, symbol Transistor_BJT:TIP120
- added R6, R7: 1k, Resistor_SMD:R_0805_2012Metric, symbol Device:R
- added R8: 15, Resistor_SMD:R_0805_2012Metric, symbol Device:R
- Q1: renamed from Q2; footprint Package_TO_SOT_THT:TO-220-3_Vertical -> Package_TO_SOT_THT:TO-220-3_Horizontal_TabDown
- Q2: renamed from Q1; footprint Package_TO_SOT_THT:TO-220-3_Vertical -> Package_TO_SOT_THT:TO-220-3_Horizontal_TabDown
- R1: renamed from R2; footprint (none) -> Resistor_SMD:R_0805_2012Metric
- R2: renamed from R3; footprint (none) -> Resistor_SMD:R_0805_2012Metric
- R3: renamed from R4; footprint (none) -> Resistor_SMD:R_0805_2012Metric
Connections:
- net +12V: now also R8.1
- net GND: now also Q4.3 (E), R7.2
- net at Q1.2 (C), Q2.2 (C): now also J2.1 (Pin_1)
- net at R1.2: now also J2.2 (Pin_2)
- net Pulse Input renamed DRIVER_PWM_1
- new net: Q3.1 (B), R6.2, R7.1
- new net: J1.1 (Pin_1), Q3.2 (C), Q4.2 (C)
- new net: Q3.3 (E), Q4.1 (B)
- new net: J1.2 (Pin_2), R8.2
- new net DRIVER_PWM_2: R6.1
