File: LEDREC.kicad_sch (KiCad schematic)
At the start: 4 parts, among them Q1 LTR-306

Commit message: Add files via upload
Parts:
- removed C1: 1 μF, symbol Device:C_Polarized_US
- removed Q1: LTR-306, LED_THT:LED_D5.0mm_Clear, symbol Sensor_Optical:BPW40
- added C7, C8: 1u, Capacitor_SMD:C_1206_3216Metric, symbol Device:C_Polarized
- added J3, J7: Conn_01x02_Pin, Connector_PinHeader_2.54mm:PinHeader_1x02_P2.54mm_Horizontal, symbol Connector:Conn_01x02_Pin
- added R10: 100k, Resistor_SMD:R_0805_2012Metric, symbol Device:R
- added R9: 270k, Resistor_SMD:R_0805_2012Metric, symbol Device:R
- R4: renamed from R2; value 120k -> 270k; footprint (none) -> Resistor_SMD:R_0805_2012Metric
- R5: renamed from R3; footprint (none) -> Resistor_SMD:R_0805_2012Metric
Connections:
- net +3.3V: now also J3.1 (Pin_1), J7.1 (Pin_1)
- net GND: now also C7.2, C8.2, R9.2
- net at R4.1, R5.1: now also J3.2 (Pin_2)
- net To PWM renamed IR_Sense_2
- net IR_Sense_2: now also C8.1
- new net: J7.2 (Pin_2), R10.1, R9.1
- new net IR_Sense_1: C7.1, R10.2
