File: rain sensor schematics.kicad_sch (KiCad schematic)
At the start: 10 parts, among them Q1 LTR-306, Q1 TIP120, Q2 TIP120

Commit message: Add files via upload
Parts:
- removed C1: 1 μF, symbol Device:C_Polarized_US
- removed D1: D, symbol Device:D
- removed Q1, Q2: TIP120, Package_TO_SOT_THT:TO-220-3_Vertical, symbol Transistor_BJT:TIP120
- removed Q1: LTR-306, LED_THT:LED_D5.0mm_Clear, symbol Sensor_Optical:BPW40
- removed R2: 15, symbol Device:R
- removed R2: 120k, symbol Device:R
- removed R3: 100k, symbol Device:R
- removed R3, R4: 1k, symbol Device:R
- added H1, H2, H3, H4: MountingHole, MountingHole:MountingHole_2.2mm_M2_ISO14580_Pad_TopBottom, symbol Mechanical:MountingHole
Other:
- added sheet CAN_MCU (untitled.kicad_sch)
- added sheet Power_conv (12v-3.3v.kicad_sch)
- sheet IR LED Driver Circuit ports: added DRIVER_PWM_1, DRIVER_PWM_2; removed none
- sheet LED Receiver Circuit ports: added IR_Sense_1, IR_Sense_2; removed none
